Commit message: Add IMU, tune cartographer, change planner to TEB

File: insnow_description/urdf/insnow.xacro (robot description, xacro)
@@ -64,4 +64,6 @@
   </collision>
 </link>
+<link name="t265_imu_optical_frame">
+</link>
 <joint name="velodyne_joint" type="fixed">
   <origin rpy="0 0 0" xyz="0.08046 0.002321 0.759661"/>
@@ -70,7 +72,12 @@
 </joint>
 <joint name="t265_joint" type="fixed">
-  <origin rpy="0 0 0" xyz="0.115584 0.000979 0.750347"/>
+  <origin rpy="0 0.015 0" xyz="0.115584 0.000979 0.750347"/>
   <parent link="base_link"/>
   <child link="t265_link"/>
 </joint>
+<joint name="t265_imu" type="fixed">
+  <origin rpy="-1.570796327 0 0" xyz="0.0 0.0 0.0"/>
+  <parent link="t265_link"/>
+  <child link="t265_imu_optical_frame"/>
+</joint>
 </robot>
